File: Testing/CAD/Pulse Gen/Pulse Gen.kicad_sch (KiCad schematic)
At the start: 15 parts, among them U1 LM393

Commit message: working magnetic core memorygit add .
Parts:
- removed C1, C2: 100m, symbol Device:C
- removed R1, R10, R3, R4, R5, R6, R9: 1k, symbol Device:R
- removed R2: 10k, symbol Device:R
- removed R7, R8: 100, symbol Device:R
- removed U1: LM393, symbol Comparator:LM393
- removed V1: 5, symbol Simulation_SPICE:VDC
- removed V2: 1, symbol Simulation_SPICE:VDC
